File: electronics/motor_driver/chargepump.sch (KiCad schematic (older format))
At the start: 15 parts, among them Q301 Q_NPN_BEC, Q302 Q_NPN_BEC, U301 NE555, U302 LM7810ACT

Commit message: Rensa + byta footprints + ändra vior + uppdatera kontakt.
Parts:
- C301: footprint Capacitors_SMD:C_0603_HandSoldering -> Capacitors_SMD:C_0805_HandSoldering
- R301, R302, R303, R304: footprint Resistors_SMD:R_0603_HandSoldering -> Resistors_SMD:R_0805_HandSoldering
Changed lines of the file:
@@
 F 0 "R301" H 3270 2096 50  0000 L CNN
 F 1 "1k" H 3270 2005 50  0000 L CNN
-F 2 "Resistors_SMD:R_0603_HandSoldering" V 3130 2050 50  0001 C CNN
+F 2 "Resistors_SMD:R_0805_HandSoldering" V 3130 2050 50  0001 C CNN
 F 3 "~" H 3200 2050 50  0001 C CNN
 	1    3200 2050
@@
 F 0 "R302" H 3270 2496 50  0000 L CNN
 F 1 "150k" H 3270 2405 50  0000 L CNN
-F 2 "Resistors_SMD:R_0603_HandSoldering" V 3130 2450 50  0001 C CNN
+F 2 "Resistors_SMD:R_0805_HandSoldering" V 3130 2450 50  0001 C CNN
 F 3 "~" H 3200 2450 50  0001 C CNN
 	1    3200 2450
@@
 F 0 "C301" H 3315 2946 50  0000 L CNN
 F 1 "1n" H 3315 2855 50  0000 L CNN
-F 2 "Capacitors_SMD:C_0603_HandSoldering" H 3238 2750 50  0001 C CNN
+F 2 "Capacitors_SMD:C_0805_HandSoldering" H 3238 2750 50  0001 C CNN
 F 3 "~" H 3200 2900 50  0001 C CNN
 	1    3200 2900
@@
 F 0 "R303" V 3393 2050 50  0000 C CNN
 F 1 "1k" V 3484 2050 50  0000 C CNN
-F 2 "Resistors_SMD:R_0603_HandSoldering" V 3530 2050 50  0001 C CNN
+F 2 "Resistors_SMD:R_0805_HandSoldering" V 3530 2050 50  0001 C CNN
 F 3 "~" H 3600 2050 50  0001 C CNN
 	1    3600 2050
@@
 F 0 "R304" H 4080 1104 50  0000 R CNN
 F 1 "1k" H 4080 1195 50  0000 R CNN
-F 2 "Resistors_SMD:R_0603_HandSoldering" V 4080 1150 50  0001 C CNN
+F 2 "Resistors_SMD:R_0805_HandSoldering" V 4080 1150 50  0001 C CNN
 F 3 "~" H 4150 1150 50  0001 C CNN
 	1    4150 1150
