File: electronics/motor_driver/single_motor_dirver.sch (KiCad schematic (older format))
At the start: 34 parts, among them J201 CONN_01X02, Q201 Q_NMOS_GDS, Q202 Q_NMOS_GDS, Q203 Q_NPN_BEC, Q204 Q_NPN_BEC, Q205 Q_NMOS_GDS, Q206 Q_NMOS_GDS, Q207 Q_NMOS_GDS, Q208 Q_NMOS_GDS, Q209 Q_NPN_BEC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

Commit message: Rensa + byta footprints + ändra vior + uppdatera kontakt.
Parts:
- C201, C203, C204: footprint Capacitors_SMD:C_0603_HandSoldering -> Capacitors_SMD:C_0805_HandSoldering
- R201, R203, R204, R205, R206, R207, R208, R209, R210, R211, R212, R215, R216, R217: footprint Resistors_SMD:R_0603_HandSoldering -> Resistors_SMD:R_0805_HandSoldering
