File: electronics/motor_driver/motor_driver.kicad_pcb (KiCad board)
At the start: 2 copper layers, 231.6 x 160 mm, 156 parts, among them J101 CONN_02X20, J102 CONN_01X02, J103 CONN_01X02, J104 CONN_01X02, J201 CONN_01X02, J401 CONN_01X02, J501 CONN_01X02, J601 CONN_01X02, Q201 Q_NMOS_GDS, Q202 Q_NMOS_GDS, Q203 Q_NPN_BEC, Q204 Q_NPN_BEC, Q205 Q_NMOS_GDS, Q206 Q_NMOS_GDS, Q207 Q_NMOS_GDS, Q208 Q_NMOS_GDS, Q209 Q_NPN_BEC, Q210 Q_NPN_BEC, Q211 Q_NMOS_GDS, Q212 Q_NMOS_GDS, Q301 Q_NPN_BEC, Q302 Q_NPN_BEC, Q401 Q_NMOS_GDS, Q402 Q_NMOS_GDS, Q403 Q_NPN_BEC, Q404 Q_NPN_BEC, Q405 Q_NMOS_GDS, Q406 Q_NMOS_GDS, Q407 Q_NMOS_GDS, Q408 Q_NMOS_GDS, Q409 Q_NPN_BEC, Q410 Q_NPN_BEC, Q411 Q_NMOS_GDS, Q412 Q_NMOS_GDS, Q501 Q_NMOS_GDS, Q502 Q_NMOS_GDS, Q503 Q_NPN_BEC, Q504 Q_NPN_BEC, Q505 Q_NMOS_GDS, Q506 Q_NMOS_GDS, Q507 Q_NMOS_GDS, Q508 Q_NMOS_GDS, Q509 Q_NPN_BEC, Q510 Q_NPN_BEC, Q511 Q_NMOS_GDS, Q512 Q_NMOS_GDS, Q601 Q_NMOS_GDS, Q602 Q_NMOS_GDS, Q603 Q_NPN_BEC, Q604 Q_NPN_BEC, Q605 Q_NMOS_GDS, Q606 Q_NMOS_GDS, Q607 Q_NMOS_GDS, Q608 Q_NMOS_GDS, Q609 Q_NPN_BEC, Q610 Q_NPN_BEC, Q611 Q_NMOS_GDS, Q612 Q_NMOS_GDS, U201 Opamp_Dual_Generic, U301 NE555, U302 LM7810ACT, U401 Opamp_Dual_Generic, U501 Opamp_Dual_Generic, U601 Opamp_Dual_Generic

Commit message: Rensa + byta footprints + ändra vior + uppdatera kontakt.
Parts:
- added C304: 47u, Capacitors_THT:CP_Radial_D5.0mm_P2.50mm, F.Cu at (337.0, 67.9)
- C201, C203, C204, C301, C401, C403, C404, C501, C503, C504, C601, C603, C604: footprint Capacitors_SMD:C_0603_HandSoldering -> Capacitors_SMD:C_0805_HandSoldering
- C302: value 100u -> 220u; moved to F.Cu
- C303: value 10u -> 220u; footprint Capacitors_THT:CP_Radial_D5.0mm_P2.00mm -> Capacitors_THT:CP_Radial_D5.0mm_P2.50mm; moved to F.Cu
- J101: value CONN_02X20 -> IDE PATA Connector
- R201, R203, R204, R205, R206, R207, R208, R209, R210, R211, R212, R215, R216, R217, R301, R302, R303, R304, R401, R403, R404, R405, R406, R407, R408, R409, R410, R411, R412, R415, R416, R417, R501, R503, R504, R505, R506, R507, R508, R509, R510, R511, R512, R515, R516, R517, R601, R603, R604, R605, R606, R607, R608, R609, R610, R611, R612, R615, R616, R617: footprint Resistors_SMD:R_0603_HandSoldering -> Resistors_SMD:R_0805_HandSoldering
- moved C303 97.2 mm to (329.6, 67.9), turned to 0 degrees
- moved C302 83.9 mm to (322.3, 67.9), turned to 0 degrees
- moved R206 54.3 mm to (285.8, 133.7)
- moved R205 54.2 mm to (288.0, 133.8)
- moved C401 53.9 mm to (158.6, 221.4)
- moved Q410 53.9 mm to (162.1, 231.4)
- moved R401 53.9 mm to (150.2, 212.8)
- moved R416 53.9 mm to (168.8, 248.2)
- moved C504 53.9 mm to (98.1, 220.9)
- moved Q403 53.9 mm to (159.1, 225.3)
- moved Q404 53.9 mm to (174.9, 240.7)
- moved Q409 53.9 mm to (173.0, 236.8)
- moved Q503 53.9 mm to (101.7, 230.9)
- moved Q509 53.9 mm to (114.4, 240.2)
- moved Q510 53.9 mm to (112.5, 236.3)
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Connections:
- C303 pad 2: GND -> Net-(C302-Pad1)
- D301 pad 2: Net-(C302-Pad1) -> Net-(C302-Pad2)
- D302 pad 1: Net-(C302-Pad2) -> Net-(C303-Pad1)
- D303 pad 1: Net-(C303-Pad1) -> Net-(C304-Pad1)
- D303 pad 2: Net-(C302-Pad2) -> Net-(C303-Pad1)
- J101 pad 10: /RPWM_3 -> /L_IS_3
- J101 pad 12: /LPWM_3 -> /R_IS_3
- J101 pad 13: (no net) -> /R_EN_1
- J101 pad 14: (no net) -> /L_EN_3
- J101 pad 15: (no net) -> /L_EN_1
- J101 pad 16: (no net) -> /R_EN_3
- J101 pad 18: /R_IS_3 -> /LPWM_3
- J101 pad 19: (no net) -> /L_IS_1
- J101 pad 20: (no net) -> /RPWM_3
- J101 pad 22: /RPWM_4 -> /L_IS_4
- J101 pad 24: /LPWM_4 -> /R_IS_4
- J101 pad 25: (no net) -> /R_EN_2
- J101 pad 26: (no net) -> /L_EN_4
- J101 pad 27: (no net) -> /L_EN_2
- J101 pad 28: (no net) -> /R_EN_4
- J101 pad 30: /R_IS_4 -> /LPWM_4
- J101 pad 31: (no net) -> /L_IS_2
- J101 pad 32: (no net) -> /RPWM_4
- Q302 pad 2: Net-(C302-Pad1) -> Net-(C302-Pad2)
- U301 pad 5: (no net) -> Net-(U301-Pad5)
- U302 pad 1: Net-(C303-Pad1) -> Net-(C304-Pad1)
Routing:
- net Net-(C304-Pad1): track 0.00 -> 26.1 mm
- net Net-(C303-Pad1): track 26.1 -> 9.33 mm
- net Net-(C302-Pad1): track 16.0 -> 0.00 mm
- net GND: track 448.8 -> 461.9 mm
- net Net-(C302-Pad2): track 9.33 -> 16.0 mm
- net /MotorDriver1/I_LOW: track 114.5 -> 109.8 mm
- net Net-(R208-Pad1): track 9.51 -> 5.62 mm
- net Net-(R206-Pad1): track 3.54 -> 0.00 mm
- net Net-(R205-Pad1): track 7.93 -> 5.20 mm
- net Net-(R202-Pad2): track 6.33 -> 8.66 mm
- net Net-(R202-Pad3): track 4.28 -> 4.91 mm
- added copper zone on F.Cu, net GND
- added copper zone on B.Cu, net VCC
Other:
- board size 231.6 x 160 mm -> 235 x 160 mm
- net class Default: trace_width 0.3 -> 1; via_dia 0.8 -> 2.5; via_drill 0.4 -> 1

Commit message: Routa sektion av kretskortet.
Parts:
- moved R517 160.6 mm to (140.5, 91.0), turned to 0 degrees
- moved Q509 156.3 mm to (145.5, 87.0), turned to 180 degrees
- moved R516 154.8 mm to (120.0, 90.2)
- moved Q510 151.2 mm to (136.8, 87.0), turned to 180 degrees
- moved U501 150.5 mm to (100.2, 91.1)
- moved R509 146.6 mm to (147.0, 91.0), turned to 0 degrees
- moved R503 146.4 mm to (117.0, 90.2)
- moved R504 146.1 mm to (134.0, 94.0), turned to 180 degrees
- moved Q503 141.5 mm to (126.0, 91.5), turned to 180 degrees
- moved D501 141.1 mm to (90.0, 82.5), turned to 90 degrees
- moved Q504 140.5 mm to (126.0, 87.0), turned to 0 degrees
- moved R506 140.4 mm to (91.2, 101.2), turned to 180 degrees
- moved R512 135.3 mm to (134.0, 91.0), turned to 180 degrees
- moved C503 133.7 mm to (91.2, 91.5), turned to 180 degrees
- moved C504 132.6 mm to (91.2, 88.5), turned to 180 degrees
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Routing:
- net VCC: track 836.0 -> 695.9 mm
- net /MotorDriver3/CW_INT: track 0.00 -> 86.1 mm, vias 0 -> 1
- net /MotorDriver3/CCW_INT: track 0.00 -> 80.5 mm, vias 0 -> 1
- net /MotorDriver3/OUT_1: track 36.2 -> 115.7 mm
- net /RPWM_3: track 0.00 -> 73.8 mm, vias 0 -> 1
- net /MotorDrvier4/I_LOW: track 107.9 -> 47.5 mm
- net /MotorDriver1/I_LOW: track 109.8 -> 55.5 mm
- net +5V: track 67.5 -> 40.3 mm
- net /LPWM_3: track 0.00 -> 26.4 mm
- net /RPWM_2: track 0.00 -> 26.4 mm
- net /MotorDriver2/CW_INT: track 0.00 -> 26.4 mm
- net /LPWM_2: track 0.00 -> 26.3 mm
- net /RPWM_4: track 0.00 -> 25.2 mm
- net /MotorDrvier4/CCW_INT: track 0.00 -> 25.2 mm
- net /MotorDriver2/CCW_INT: track 0.00 -> 25.2 mm
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- added copper zone on B.Cu, net +5V

Commit message: Fortsätt routa logik.
Parts:
- moved R415 228.9 mm to (-11.0, 112.0), turned to 0 degrees
- moved U401 222.1 mm to (-2.00, 118.0)
- moved D401 211.2 mm to (-13.0, 108.0), turned to 90 degrees
- moved C404 204.3 mm to (-11.0, 116.0), turned to 180 degrees
- moved R410 199.2 mm to (-11.0, 122.0), turned to 180 degrees
- moved Q404 198.9 mm to (7.00, 134.0)
- moved R411 197.9 mm to (19.5, 120.5), turned to 0 degrees
- moved R407 193.2 mm to (7.00, 120.0), turned to 180 degrees
- moved R416 191.2 mm to (13.0, 137.3)
- moved Q409 189.4 mm to (25.0, 118.6), turned to 180 degrees
- moved C401 186.2 mm to (7.25, 113.0), turned to 0 degrees
- moved R417 186.1 mm to (29.0, 118.0)
- moved R408 185.7 mm to (-11.0, 126.0), turned to 0 degrees
- moved C403 185.2 mm to (-11.0, 119.0), turned to 180 degrees
- moved R403 183.5 mm to (23.0, 135.0)
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Routing:
- net Net-(R408-Pad1): track 0.00 -> 23.6 mm
- net GND: track 446.7 -> 465.5 mm
- net Net-(R406-Pad1): track 0.00 -> 16.5 mm
- net Net-(C403-Pad1): track 0.00 -> 10.8 mm
- net Net-(Q409-Pad1): track 0.00 -> 8.46 mm
- net Net-(R415-Pad2): track 0.00 -> 8.24 mm
- net Net-(R405-Pad1): track 0.00 -> 7.51 mm
- net VCC: track 695.9 -> 702.7 mm
- net Net-(Q503-Pad1): track 8.91 -> 3.32 mm
- net /MotorDriver3/CW_INT: track 86.1 -> 80.8 mm
- net /R_IS_2: track 0.00 -> 4.27 mm
- net Net-(Q409-Pad3): track 0.00 -> 4.18 mm
- net Net-(Q504-Pad1): track 6.49 -> 4.79 mm
- net Net-(Q503-Pad3): track 8.00 -> 7.48 mm
Other:
- board size 235 x 160 mm -> 260 x 160 mm

Commit message: Routa lokala nät.
Parts:
- C201, C203, C204, C601, C603, C604, D201, Q203, Q204, Q209, Q210, R201, R203, R204, R205, R206, R207, R208, R209, R210, R211, R212, R215, R216, R217, R605, R606, R607, R608, R610, R615, U201, U601: moved to F.Cu
- D601: moved to B.Cu
- moved R605 228.3 mm to (481.0, 91.0), turned to 0 degrees
- moved R607 220.8 mm to (481.0, 88.0), turned to 180 degrees
- moved C601 215.6 mm to (481.0, 85.0), turned to 0 degrees
- moved U601 214.0 mm to (473.5, 81.5), turned to 270 degrees
- moved R610 203.9 mm to (464.9, 85.5), turned to 180 degrees
- moved R606 201.4 mm to (464.9, 92.5), turned to 180 degrees
- moved C604 197.9 mm to (464.9, 82.5), turned to 180 degrees
- moved D601 194.6 mm to (463.5, 73.0), turned to 0 degrees
- moved R608 194.3 mm to (464.9, 89.5), turned to 0 degrees
- moved R615 193.1 mm to (464.9, 76.5), turned to 0 degrees
- moved C603 189.9 mm to (464.9, 79.5), turned to 180 degrees
- moved D401 182.2 mm to (169.0, 100.0), turned to 0 degrees
- moved C403 181.7 mm to (170.5, 109.5)
- moved C404 181.7 mm to (170.5, 106.5)
- moved R408 181.7 mm to (170.5, 116.5)
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Routing:
- net /RPWM_1: track 103.9 -> 25.5 mm, vias 1 -> 0
- net /MotorDriver2/CCW_INT: track 25.2 -> 73.5 mm, vias 0 -> 1
- net /RPWM_2: track 26.4 -> 73.8 mm, vias 0 -> 1
- net /MotorDriver2/CW_INT: track 26.4 -> 69.5 mm, vias 0 -> 1
- net Net-(R502-Pad2): track 0.00 -> 39.4 mm
- net /LPWM_3: track 26.4 -> 63.7 mm, vias 0 -> 1
- net /LPWM_2: track 26.3 -> 62.8 mm, vias 0 -> 1
- net /MotorDriver1/CCW_INT: track 62.0 -> 29.3 mm
- net GND: track 465.5 -> 434.8 mm
- net Net-(R402-Pad2): track 0.00 -> 30.2 mm
- net Net-(R608-Pad1): track 0.00 -> 20.2 mm
- net Net-(R502-Pad3): track 0.00 -> 19.4 mm
- net Net-(R606-Pad1): track 0.00 -> 17.3 mm
- net Net-(R206-Pad1): track 0.00 -> 17.0 mm
- net /RPWM_3: track 73.8 -> 57.4 mm
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
Commit message: Majoritet färdigt
Parts:
- moved C601 206.8 mm to (276.0, 112.0)
- moved C603 206.8 mm to (259.9, 106.5)
- moved C604 206.8 mm to (259.9, 109.5)
- moved D601 206.8 mm to (258.5, 100.0)
- moved R605 206.8 mm to (276.0, 118.0)
- moved R606 206.8 mm to (259.9, 119.5)
- moved R607 206.8 mm to (276.0, 115.0)
- moved R608 206.8 mm to (259.9, 116.5)
- moved R610 206.8 mm to (259.9, 112.5)
- moved R615 206.8 mm to (259.9, 103.5)
- moved U601 206.8 mm to (268.5, 108.5)
- moved C201 161.5 mm to (310.0, 110.5)
- moved C203 161.5 mm to (294.8, 103.5)
- moved C204 161.5 mm to (294.8, 106.5)
- moved D201 161.5 mm to (293.5, 97.0)
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Routing:
- net /VCC_2: track 28.6 -> 371.0 mm, vias 0 -> 11
- net /LPWM_4: track 25.2 -> 279.5 mm, vias 0 -> 4
- net /RPWM_4: track 25.2 -> 240.3 mm, vias 0 -> 2
- net /LPWM_3: track 63.7 -> 260.5 mm, vias 1 -> 2
- net /RPWM_3: track 57.4 -> 217.3 mm, vias 1 -> 2
- net /R_IS_4: track 3.53 -> 139.2 mm, vias 0 -> 1
- net /RPWM_1: track 25.5 -> 148.8 mm, vias 0 -> 2
- net /R_IS_3: track 3.93 -> 118.7 mm
- net /RPWM_2: track 73.8 -> 177.3 mm, vias 1 -> 2
- net /LPWM_1: track 33.7 -> 120.4 mm, vias 0 -> 2
- net /LPWM_2: track 62.8 -> 143.5 mm, vias 1 -> 2
- net /MotorDrvier4/I_LOW: track 47.5 -> 107.1 mm, vias 0 -> 2
- net /MotorDriver3/I_LOW: track 47.5 -> 103.5 mm
- net /MotorDriver2/I_LOW: track 47.5 -> 99.0 mm
- net GND: track 434.8 -> 384.4 mm, vias 0 -> 1
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