File: electronics/styrenhet/styrenhet.kicad_pcb (KiCad board)
At the start: 2 copper layers, 160 x 100 mm, 50 parts, among them J1 12V Fan, J2 Battery_In, J3 Battery to MCU, J4 12V Fan, J5 IDE PATA Connector, J6 Motor1_In, J7 Motor2_In, J8 Motor3_In, J9 Motor4_In, U1 motor_driver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

Commit message: Ska etsa...
Parts:
- removed C1, C2, C3, C4: CP, Capacitors_THT:CP_Radial_D22.0mm_P10.00mm_SnapIn
- removed J6: Motor1_In, TerminalBlocks_Phoenix:TerminalBlock_Phoenix_MKDS1.5-2pol
- removed J7: Motor2_In, TerminalBlocks_Phoenix:TerminalBlock_Phoenix_MKDS1.5-2pol
- removed J8: Motor3_In, TerminalBlocks_Phoenix:TerminalBlock_Phoenix_MKDS1.5-2pol
- removed J9: Motor4_In, TerminalBlocks_Phoenix:TerminalBlock_Phoenix_MKDS1.5-2pol
- C10, C11, C12, C5, C6, C7, C8, C9: moved to B.Cu
- moved F1 236.1 mm to (77.0, 62.0), turned to 180 degrees
- moved J1 221.8 mm to (61.4, 55.0), turned to 90 degrees
- moved J4 215.5 mm to (74.0, 55.0), turned to 90 degrees
- moved C17 101.0 mm to (139.5, 68.5), turned to 180 degrees
- moved C20 9.71 mm to (165.5, 131.5)
- moved C18 9.60 mm to (101.5, 132.0), turned to 0 degrees
- moved C13 5.50 mm to (163.5, 103.0)
- moved C19 4.03 mm to (106.5, 68.5)
- moved C9 3.54 mm to (101.0, 83.5)
- moved C10 3.50 mm to (101.0, 109.5)
- moved C11 3.50 mm to (116.0, 115.0)
- moved C12 3.50 mm to (116.0, 90.5)
- moved C14 3.50 mm to (108.5, 96.8)
- moved C15 3.50 mm to (161.5, 97.0)
- moved C16 3.50 mm to (108.5, 103.2)
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Connections:
- U1 pad 11: /motor1+ -> Net-(U1-Pad11)
- U1 pad 12: /motor1- -> Net-(U1-Pad12)
- U2 pad 11: /motor2+ -> Net-(U2-Pad11)
- U2 pad 12: /motor2- -> Net-(U2-Pad12)
- U3 pad 11: /motor3+ -> Net-(U3-Pad11)
- U3 pad 12: /motor3- -> Net-(U3-Pad12)
- U4 pad 11: /motor4+ -> Net-(U4-Pad11)
- U4 pad 12: /motor4- -> Net-(U4-Pad12)
Routing:
- net GND: track 79.1 -> 251.5 mm, vias 0 -> 7
- net /BAT_+: track 0.00 -> 84.9 mm, vias 0 -> 4
- net Net-(F1-Pad1): track 0.00 -> 29.6 mm
- net /R_IS_4: track 153.3 -> 129.6 mm, vias 0 -> 1
- net /L_IS_4: track 188.6 -> 165.3 mm
- net /L_EN_4: track 153.8 -> 136.4 mm
- net /R_EN_4: track 128.4 -> 113.6 mm
- net /R_IS_3: track 134.1 -> 148.2 mm, vias 0 -> 1
- net /LPWM_4: track 132.5 -> 120.0 mm
- net /RPWM_4: track 109.6 -> 99.5 mm
- net /RPWM_1: track 75.4 -> 68.0 mm
- net /LPWM_1: track 107.7 -> 102.4 mm
- net /LPWM_2: track 25.2 -> 20.4 mm
- net /L_IS_3: track 152.1 -> 156.6 mm
- net /R_IS_1: track 57.3 -> 53.0 mm, vias 0 -> 1
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- added copper zone on B.Cu, net /BAT_+
Other:
- net class Power: via_dia 0.8 -> 3; via_drill 0.4 -> 1
