File: electronics/styrenhet/styrenhet.sch (KiCad schematic (older format))
At the start: 44 parts, among them J1 Screw_Terminal_01x02, J2 Screw_Terminal_01x02, J3 Screw_Terminal_01x02, J4 Screw_Terminal_01x02, J5 Screw_Terminal_01x02, J6 Screw_Terminal_01x02, J7 IDE PATA Connector, J8 12V Fan, J9 12V Fan, U1 motor_driver, U2 motor_driver, U3 motor_driver, U4 motor_driver

Commit message: Ändra maaassa grejer.
Parts:
- removed C1, C2: CP, Capacitor_THT:CP_Radial_D22.0mm_P10.00mm_SnapIn, symbol Device:CP
- removed C? (x7): 1uF, symbol Device:C
- removed J6: Screw_Terminal_01x02, TerminalBlock:TerminalBlock_bornier-2_P5.08mm, symbol Connector:Screw_Terminal_01x02
- removed R? (x7): 10k, symbol Device:R
- removed R? (x7): 1.5k, symbol Device:R
- added C1, C2, C7, C8: CP, Capacitors_THT:CP_Axial_L30.0mm_D15.0mm_P35.00mm_Horizontal, symbol Device:C
- added C17, C18, C19, C20: CP, symbol Device:CP
- added C? (x7): 47uF, symbol Device:CP
- added J6: Battery to MCU, symbol Connector:Screw_Terminal_01x01
- added R? (x7): 440R, symbol Device:R
- added R? (x7): 660R, symbol Device:R
- C9: renamed from C?; value 1uF -> 47uF; symbol Device:C -> Device:CP
- J1: value Screw_Terminal_01x02 -> Battery_In
- J2: value Screw_Terminal_01x02 -> Motor1_In
- J3: value Screw_Terminal_01x02 -> Motor2_In
- J4: value Screw_Terminal_01x02 -> Motor3_In
- J5: value Screw_Terminal_01x02 -> Motor4_In
- R1: renamed from R?; value 10k -> 660R
- R9: renamed from R?; value 1.5k -> 440R
- gave numbers to parts that had none: 1
Connections:
- net BAT_+: now also U1.10 (B+), U2.10 (B+), U3.10 (B+), U4.10 (B+), C17.1, C18.1, C19.1, C20.1; no longer J2.1 (Pin_1), J3.1 (Pin_1), J4.1 (Pin_1), J5.1 (Pin_1), J7.7 (Pin_7), J7.8 (Pin_8)
- net GND: now also J7.33 (Pin_33), J7.34 (Pin_34), U1.9 (B-), U2.9 (B-), U3.9 (B-), U4.9 (B-), C17.2, C18.2, C19.2, C20.2, C?.2, C?.2, C?.2, C?.2, C?.2, C?.2, C?.2, R?.1, R?.1, R?.1, R?.1, R?.1, R?.1, R?.1; no longer J2.2 (Pin_2), J3.2 (Pin_2), J4.2 (Pin_2), J5.2 (Pin_2), J7.10 (Pin_10), J7.9 (Pin_9)
- net LPWM_1: now also J7.11 (Pin_11); no longer J7.13 (Pin_13)
- net LPWM_2: now also J7.23 (Pin_23); no longer J7.25 (Pin_25)
- net LPWM_3: now also J7.18 (Pin_18); no longer J7.20 (Pin_20)
- net LPWM_4: now also J7.30 (Pin_30); no longer J7.32 (Pin_32)
- net L_EN_1: now also J7.15 (Pin_15); no longer J7.17 (Pin_17)
- net L_EN_2: now also J7.27 (Pin_27); no longer J7.29 (Pin_29)
- net L_EN_3: now also J7.14 (Pin_14); no longer J7.16 (Pin_16)
- net L_EN_4: now also J7.26 (Pin_26); no longer J7.28 (Pin_28)
- net L_IS_1: now also J7.19 (Pin_19), C?.1, R?.2, R?.2; no longer J7.21 (Pin_21)
- net L_IS_2: now also J7.31 (Pin_31), C?.1, R?.2, R?.2; no longer J7.33 (Pin_33)
- net L_IS_3: now also J7.10 (Pin_10), C?.1, R?.2, R?.2; no longer J7.12 (Pin_12)
- net L_IS_4: now also J7.22 (Pin_22), C?.1, R?.2, R?.2; no longer J7.24 (Pin_24)
- net RPWM_1: now also J7.9 (Pin_9); no longer J7.11 (Pin_11)
- net RPWM_2: now also J7.21 (Pin_21); no longer J7.23 (Pin_23)
- net RPWM_3: now also J7.20 (Pin_20); no longer J7.22 (Pin_22)
- net RPWM_4: now also J7.32 (Pin_32); no longer J7.34 (Pin_34)
- net R_EN_1: now also J7.13 (Pin_13); no longer J7.15 (Pin_15)
- net R_EN_2: now also J7.25 (Pin_25); no longer J7.27 (Pin_27)
- net R_EN_3: now also J7.16 (Pin_16); no longer J7.18 (Pin_18)
- net R_EN_4: now also J7.28 (Pin_28); no longer J7.30 (Pin_30)
- net R_IS_1: now also J7.17 (Pin_17), R9.2; no longer J7.19 (Pin_19)
- net R_IS_2: now also J7.29 (Pin_29), C?.1, R?.2, R?.2; no longer J7.31 (Pin_31)
- net R_IS_3: now also J7.12 (Pin_12), C?.1, R?.2, R?.2; no longer J7.14 (Pin_14)
- net R_IS_4: now also J7.24 (Pin_24), C?.1, R?.2, R?.2; no longer J7.26 (Pin_26)
- net motor1+: now reaches U1.11 (M+)
- net motor1+: now also J2.1 (Pin_1), C1.1
- net motor1-: now reaches U1.12 (M-)
- net motor1-: now also J2.2 (Pin_2), C1.2
- net at U1.6 (L_IS): now also R?.1
- net motor2+: now reaches U2.11 (M+)
- net motor2+: now also J3.1 (Pin_1), C2.1
- net motor2-: now reaches U2.12 (M-)
- net motor2-: now also J3.2 (Pin_2), C2.2
- net at U2.6 (L_IS): now also R?.1
- net motor3+: now reaches U3.11 (M+)
- net motor3+: now also J4.1 (Pin_1), C7.1
- net motor3-: now reaches U3.12 (M-)
- net motor3-: now also J4.2 (Pin_2), C7.2
- net at U3.6 (L_IS): now also R?.1
- net motor4+: now reaches U4.11 (M+)
- net motor4+: now also J5.1 (Pin_1), C8.1
- net motor4-: now reaches U4.12 (M-)
- net motor4-: now also J5.2 (Pin_2), C8.2
- net at U4.6 (L_IS): now also R?.1
- new net: R1.1, U1.5 (VCC)
- new net: R?.1, U2.5 (VCC)
- new net: R?.1, U3.5 (VCC)
- new net: R?.1, U4.5 (VCC)
- new net B_MCU: J6.1 (Pin_1), J7.7 (Pin_7), J7.8 (Pin_8)
Other:
- note added: "Battery in to MCU-kort\n\n"
- note added: "Battery in\n"
- note added: "Motor connectors\n"
- note added: "Note: On separate in line fuse."
- note removed: "Note: 1.5k resistor value is not confirmed.\n"
- moved on the sheet: C3, C4, C5, C6, J1, J2, J3, J4, J5, R1, R9, U1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

Commit message: Finish schematic:
Parts:
- C1, C2: footprint Capacitors_THT:CP_Axial_L30.0mm_D15.0mm_P35.00mm_Horizontal -> Capacitors_THT:CP_Radial_D22.0mm_P10.00mm_SnapIn
- C10, C11, C12, C6, C7, C8, C9: renamed from C?; footprint (none) -> Capacitors_THT:CP_Radial_D10.0mm_P5.00mm
- C13: renamed from C3; footprint Capacitor_SMD:C_1206_3216Metric_Pad1.42x1.75mm_HandSolder -> Capacitors_SMD:C_0805_HandSoldering
- C14: renamed from C4; footprint Capacitor_SMD:C_1206_3216Metric_Pad1.42x1.75mm_HandSolder -> Capacitors_SMD:C_0805_HandSoldering
- C15: renamed from C5; footprint Capacitor_SMD:C_1206_3216Metric_Pad1.42x1.75mm_HandSolder -> Capacitors_SMD:C_0805_HandSoldering
- C16: renamed from C6; footprint Capacitor_SMD:C_1206_3216Metric_Pad1.42x1.75mm_HandSolder -> Capacitors_SMD:C_0805_HandSoldering
- C17, C18, C19, C20: footprint (none) -> Capacitors_THT:CP_Radial_D22.0mm_P10.00mm_SnapIn
- C3: renamed from C7; footprint Capacitors_THT:CP_Axial_L30.0mm_D15.0mm_P35.00mm_Horizontal -> Capacitors_THT:CP_Radial_D22.0mm_P10.00mm_SnapIn
- C4: renamed from C8; footprint Capacitors_THT:CP_Axial_L30.0mm_D15.0mm_P35.00mm_Horizontal -> Capacitors_THT:CP_Radial_D22.0mm_P10.00mm_SnapIn
- C5: renamed from C9; footprint (none) -> Capacitors_THT:CP_Radial_D10.0mm_P5.00mm
- F1: footprint styrenhet-footprints:SMD_Fuse_holder -> styrenhet-footprints:ETA_thl_fuseholder
- J1: renamed from J8; footprint (none) -> Pin_Headers:Pin_Header_Straight_1x04_Pitch2.54mm
- J3: renamed from J6; footprint (none) -> TerminalBlocks_Phoenix:TerminalBlock_Phoenix_MKDS1.5-2pol
- J4: renamed from J9; footprint (none) -> Pin_Headers:Pin_Header_Straight_1x04_Pitch2.54mm
- R1: renamed from R9; footprint (none) -> Resistors_SMD:R_0603_HandSoldering
- R10, R11, R12, R13, R14, R15, R16, R2, R3, R4, R5, R6, R7, R8: renamed from R?; footprint (none) -> Resistors_SMD:R_0603_HandSoldering
- R9: renamed from R1; footprint (none) -> Resistors_SMD:R_0603_HandSoldering
- renumbered J1 to J2, J7 to J5, J2 to J6, J3 to J7, J4 to J8, J5 to J9

Commit message: Uppdatera footprints.
Parts:
- J3: symbol Connector:Screw_Terminal_01x01 -> Connector:Screw_Terminal_01x02
- J6, J7, J8, J9: footprint TerminalBlock:TerminalBlock_bornier-2_P5.08mm -> TerminalBlocks_Phoenix:TerminalBlock_Phoenix_MKDS1.5-2pol
Connections:
- net B_MCU: now also J3.2 (Pin_2)
Changed lines of the file:
@@
 F 0 "J9" V 6316 1162 50  0000 R CNN
 F 1 "Motor4_In" V 6225 1162 50  0000 R CNN
-F 2 "TerminalBlock:TerminalBlock_bornier-2_P5.08mm" H 6350 1350 50  0001 C CNN
+F 2 "TerminalBlocks_Phoenix:TerminalBlock_Phoenix_MKDS1.5-2pol" H 6350 1350 50  0001 C CNN
 F 3 "~" H 6350 1350 50  0001 C CNN
 	1    6350 1350
@@
 F 0 "J8" V 5616 1162 50  0000 R CNN
 F 1 "Motor3_In" V 5525 1162 50  0000 R CNN
-F 2 "TerminalBlock:TerminalBlock_bornier-2_P5.08mm" H 5650 1350 50  0001 C CNN
+F 2 "TerminalBlocks_Phoenix:TerminalBlock_Phoenix_MKDS1.5-2pol" H 5650 1350 50  0001 C CNN
 F 3 "~" H 5650 1350 50  0001 C CNN
 	1    5650 1350
@@
 F 0 "J7" V 4916 1162 50  0000 R CNN
 F 1 "Motor2_In" V 4825 1162 50  0000 R CNN
-F 2 "TerminalBlock:TerminalBlock_bornier-2_P5.08mm" H 4950 1350 50  0001 C CNN
+F 2 "TerminalBlocks_Phoenix:TerminalBlock_Phoenix_MKDS1.5-2pol" H 4950 1350 50  0001 C CNN
 F 3 "~" H 4950 1350 50  0001 C CNN
 	1    4950 1350
@@
 F 0 "J6" V 4216 1162 50  0000 R CNN
 F 1 "Motor1_In" V 4125 1162 50  0000 R CNN
-F 2 "TerminalBlock:TerminalBlock_bornier-2_P5.08mm" H 4250 1350 50  0001 C CNN
+F 2 "TerminalBlocks_Phoenix:TerminalBlock_Phoenix_MKDS1.5-2pol" H 4250 1350 50  0001 C CNN
 F 3 "~" H 4250 1350 50  0001 C CNN
 	1    4250 1350
@@
 Battery in to MCU-kort\n\n
 $Comp
-L Connector:Screw_Terminal_01x01 J3
+L Connector:Screw_Terminal_01x02 J3
 U 1 1 5D3EBD49
 P 1850 5250
-F 0 "J3" H 1768 5025 50  0000 C CNN
-F 1 "Battery to MCU" H 1768 5116 50  0000 C CNN
+F 0 "J3" H 1850 5050 50  0000 C CNN
+F 1 "Battery to MCU" H 2050 5350 50  0000 C CNN
 F 2 "TerminalBlocks_Phoenix:TerminalBlock_Phoenix_MKDS1.5-2pol" H 1850 5250 50  0001 C CNN
 F 3 "~" H 1850 5250 50  0001 C CNN
@@
 	-1   0    0    1
 $EndComp
-Text Label 2450 5250 2    50   ~ 0
+Text Label 2450 5200 2    50   ~ 0
 B_MCU
-Wire Wire Line
-	2450 5250 2050 5250
 Wire Notes Line
 	1150 4550 1150 5450
@@
 	11100 8650 11400 8650
 Connection ~ 11400 8650
+Wire Wire Line
+	2050 5150 2100 5150
+Wire Wire Line
+	2100 5150 2100 5200
+Wire Wire Line
+	2100 5200 2450 5200
+Wire Wire Line
+	2050 5250 2100 5250
+Wire Wire Line
+	2100 5250 2100 5200
+Connection ~ 2100 5200
 $EndSCHEMATC
