File: electronics/styrenhet/styrenhet.sch (KiCad schematic (older format))
At the start: 50 parts, among them J1 12V Fan, J2 Battery_In, J3 Battery to MCU, J4 12V Fan, J5 IDE PATA Connector, J6 Motor1_In, J7 Motor2_In, J8 Motor3_In, J9 Motor4_In, U1 motor_driver, U2 motor_driver, U3 motor_driver, U4 motor_driver

Commit message: Add IDE PATA footprint.
Parts:
- J5: footprint Connector_IDC:IDC-Header_2x20_P2.54mm_Vertical -> styrenhet-footprints:IDC-Header_2x20_Pitch2.54mm_Straight
Changed lines of the file:
@@
 Wire Wire Line
 	12600 2750 12600 2800
-Text Label 12600 1800 0    50   ~ 6
+Text Label 12600 1800 0    50   ~ 10
 RPWM_1
 Wire Wire Line
 	12600 1800 13250 1800
-Text Label 12600 1900 0    50   ~ 6
+Text Label 12600 1900 0    50   ~ 10
 LPWM_1
 Wire Wire Line
 	12600 1900 13250 1900
-Text Label 12600 2000 0    50   ~ 6
+Text Label 12600 2000 0    50   ~ 10
 R_EN_1
-Text Label 12600 2100 0    50   ~ 6
+Text Label 12600 2100 0    50   ~ 10
 L_EN_1
-Text Label 11100 1550 0    50   ~ 6
+Text Label 11100 1550 0    50   ~ 10
 R_IS_1
 Wire Wire Line
@@
 Wire Wire Line
 	12600 4800 12600 4850
-Text Label 12600 3850 0    50   ~ 6
+Text Label 12600 3850 0    50   ~ 10
 RPWM_2
 Wire Wire Line
 	12600 3850 13250 3850
-Text Label 12600 3950 0    50   ~ 6
+Text Label 12600 3950 0    50   ~ 10
 LPWM_2
 Wire Wire Line
 	12600 3950 13250 3950
-Text Label 12600 4050 0    50   ~ 6
+Text Label 12600 4050 0    50   ~ 10
 R_EN_2
-Text Label 12600 4150 0    50   ~ 6
+Text Label 12600 4150 0    50   ~ 10
 L_EN_2
-Text Label 11100 3600 0    50   ~ 6
+Text Label 11100 3600 0    50   ~ 10
 R_IS_2
-Text Label 11100 4600 0    50   ~ 6
+Text Label 11100 4600 0    50   ~ 10
 L_IS_2
 Wire Wire Line
@@
 Wire Wire Line
 	12600 6850 12600 6900
-Text Label 12600 5900 0    50   ~ 6
+Text Label 12600 5900 0    50   ~ 10
 RPWM_3
 Wire Wire Line
 	12600 5900 13250 5900
-Text Label 12600 6000 0    50   ~ 6
+Text Label 12600 6000 0    50   ~ 10
 LPWM_3
 Wire Wire Line
 	12600 6000 13250 6000
-Text Label 12600 6100 0    50   ~ 6
+Text Label 12600 6100 0    50   ~ 10
 R_EN_3
-Text Label 12600 6200 0    50   ~ 6
+Text Label 12600 6200 0    50   ~ 10
 L_EN_3
-Text Label 11100 5650 0    50   ~ 6
+Text Label 11100 5650 0    50   ~ 10
 R_IS_3
-Text Label 11100 6650 0    50   ~ 6
+Text Label 11100 6650 0    50   ~ 10
 L_IS_3
 Wire Wire Line
@@
 Wire Wire Line
 	12600 8950 12600 9000
-Text Label 12600 8000 0    50   ~ 6
+Text Label 12600 8000 0    50   ~ 10
 RPWM_4
 Wire Wire Line
 	12600 8000 13250 8000
-Text Label 12600 8100 0    50   ~ 6
+Text Label 12600 8100 0    50   ~ 10
 LPWM_4
 Wire Wire Line
 	12600 8100 13250 8100
-Text Label 12600 8200 0    50   ~ 6
+Text Label 12600 8200 0    50   ~ 10
 R_EN_4
-Text Label 12600 8300 0    50   ~ 6
+Text Label 12600 8300 0    50   ~ 10
 L_EN_4
-Text Label 11100 7650 0    50   ~ 6
+Text Label 11100 7650 0    50   ~ 10
 R_IS_4
-Text Label 11100 8650 0    50   ~ 6
+Text Label 11100 8650 0    50   ~ 10
 L_IS_4
 Wire Wire Line
@@
 	0    1    1    0
 $EndComp
-Text Label 2250 2450 1    50   ~ 6
+Text Label 2250 2450 1    50   ~ 10
 BAT_+
 Wire Wire Line
@@
 F 0 "J5" H 3000 10167 50  0000 C CNN
 F 1 "IDE PATA Connector" H 3000 10076 50  0000 C CNN
-F 2 "Connector_IDC:IDC-Header_2x20_P2.54mm_Vertical" H 2950 9050 50  0001 C CNN
+F 2 "styrenhet-footprints:IDC-Header_2x20_Pitch2.54mm_Straight" H 2950 9050 50  0001 C CNN
 F 3 "~" H 2950 9050 50  0001 C CNN
 	1    2950 9050
@@
 Wire Wire Line
 	2600 10050 2600 10250
-Text Label 3900 9050 2    50   ~ 6
+Text Label 3900 9050 2    50   ~ 10
 RPWM_3
 Wire Wire Line
 	3900 9050 3250 9050
-Text Label 3900 8950 2    50   ~ 6
+Text Label 3900 8950 2    50   ~ 10
 LPWM_3
 Wire Wire Line
 	3900 8950 3250 8950
-Text Label 3900 8850 2    50   ~ 6
+Text Label 3900 8850 2    50   ~ 10
 R_EN_3
-Text Label 3900 8750 2    50   ~ 6
+Text Label 3900 8750 2    50   ~ 10
 L_EN_3
-Text Label 3900 8650 2    50   ~ 6
+Text Label 3900 8650 2    50   ~ 10
 R_IS_3
-Text Label 3900 8550 2    50   ~ 6
+Text Label 3900 8550 2    50   ~ 10
 L_IS_3
 Wire Wire Line
@@
 Wire Wire Line
 	3250 8850 3900 8850
-Text Label 2100 8550 0    50   ~ 6
+Text Label 2100 8550 0    50   ~ 10
 RPWM_1
 Wire Wire Line
 	2100 8550 2750 8550
-Text Label 2100 8650 0    50   ~ 6
+Text Label 2100 8650 0    50   ~ 10
 LPWM_1
 Wire Wire Line
 	2100 8650 2750 8650
-Text Label 2100 8750 0    50   ~ 6
+Text Label 2100 8750 0    50   ~ 10
 R_EN_1
-Text Label 2100 8850 0    50   ~ 6
+Text Label 2100 8850 0    50   ~ 10
 L_EN_1
-Text Label 2100 8950 0    50   ~ 6
+Text Label 2100 8950 0    50   ~ 10
 R_IS_1
-Text Label 2100 9050 0    50   ~ 6
+Text Label 2100 9050 0    50   ~ 10
 L_IS_1
 Wire Wire Line
@@
 Wire Wire Line
 	2750 8750 2100 8750
-Text Label 2000 9150 0    50   ~ 6
+Text Label 2000 9150 0    50   ~ 10
 RPWM_2
-Text Label 2000 9250 0    50   ~ 6
+Text Label 2000 9250 0    50   ~ 10
 LPWM_2
-Text Label 2000 9350 0    50   ~ 6
+Text Label 2000 9350 0    50   ~ 10
 R_EN_2
-Text Label 2000 9450 0    50   ~ 6
+Text Label 2000 9450 0    50   ~ 10
 L_EN_2
-Text Label 2000 9550 0    50   ~ 6
+Text Label 2000 9550 0    50   ~ 10
 R_IS_2
-Text Label 2000 9650 0    50   ~ 6
+Text Label 2000 9650 0    50   ~ 10
 L_IS_2
-Text Label 4000 9650 2    50   ~ 6
+Text Label 4000 9650 2    50   ~ 10
 RPWM_4
-Text Label 4000 9550 2    50   ~ 6
+Text Label 4000 9550 2    50   ~ 10
 LPWM_4
-Text Label 4000 9450 2    50   ~ 6
+Text Label 4000 9450 2    50   ~ 10
 R_EN_4
-Text Label 4000 9350 2    50   ~ 6
+Text Label 4000 9350 2    50   ~ 10
 L_EN_4
-Text Label 4000 9250 2    50   ~ 6
+Text Label 4000 9250 2    50   ~ 10
 R_IS_4
-Text Label 4000 9150 2    50   ~ 6
+Text Label 4000 9150 2    50   ~ 10
 L_IS_4
 Wire Wire Line
@@
 Wire Wire Line
 	3250 9150 4000 9150
-Text Notes 1700 7750 0    50   ~ 6
+Text Notes 1700 7750 0    50   ~ 10
 Note: Same pinout on both boards\n\n
 $Comp
@@
 Wire Wire Line
 	12400 8500 13250 8500
-Text Notes 12350 1100 0    79   ~ 6
+Text Notes 12350 1100 0    79   ~ 16
 Motor drivers model: BTS7960b\nResistors are for current sensing.\n
 Text Notes 1300 7950 0    157  ~ 31
@@
 Wire Notes Line
 	3450 800  1150 800
-Text Notes 1900 1100 0    79   ~ 6
+Text Notes 1900 1100 0    79   ~ 16
 Generic 12V server fans.\n
 $Comp
@@
 Wire Wire Line
 	2250 2150 2250 2450
-Text Label 14650 3950 2    50   ~ 6
+Text Label 14650 3950 2    50   ~ 10
 motor2+
-Text Label 14650 3850 2    50   ~ 6
+Text Label 14650 3850 2    50   ~ 10
 motor2-
 Wire Wire Line
@@
 Wire Wire Line
 	14150 3950 14650 3950
-Text Label 14650 6000 2    50   ~ 6
+Text Label 14650 6000 2    50   ~ 10
 motor3+
-Text Label 14650 5900 2    50   ~ 6
+Text Label 14650 5900 2    50   ~ 10
 motor3-
 Wire Wire Line
@@
 Wire Wire Line
 	14150 6000 14650 6000
-Text Label 14650 8100 2    50   ~ 6
+Text Label 14650 8100 2    50   ~ 10
 motor4+
-Text Label 14650 8000 2    50   ~ 6
+Text Label 14650 8000 2    50   ~ 10
 motor4-
 Wire Wire Line
@@
 	1    0    0    -1
 $EndComp
-Text Label 14800 2000 2    50   ~ 6
+Text Label 14800 2000 2    50   ~ 10
 BAT_+
 $Comp
@@
 	-1   0    0    -1
 $EndComp
-Text Label 2400 3650 2    50   ~ 6
+Text Label 2400 3650 2    50   ~ 10
 BAT_+
-Text Label 2400 3750 2    50   ~ 6
+Text Label 2400 3750 2    50   ~ 10
 BAT_-
 Wire Wire Line
@@
 Wire Wire Line
 	6200 2000 6200 2450
-Text Label 6600 2450 1    50   ~ 6
+Text Label 6600 2450 1    50   ~ 10
 motor4-
-Text Label 6200 2450 1    50   ~ 6
+Text Label 6200 2450 1    50   ~ 10
 motor4+
 Wire Wire Line
@@
 Wire Wire Line
 	5500 2000 5500 2450
-Text Label 5900 2450 1    50   ~ 6
+Text Label 5900 2450 1    50   ~ 10
 motor3-
-Text Label 5500 2450 1    50   ~ 6
+Text Label 5500 2450 1    50   ~ 10
 motor3+
 Wire Wire Line
@@
 Wire Wire Line
 	4800 2000 4800 2450
-Text Label 5200 2450 1    50   ~ 6
+Text Label 5200 2450 1    50   ~ 10
 motor2-
-Text Label 4800 2450 1    50   ~ 6
+Text Label 4800 2450 1    50   ~ 10
 motor2+
 Connection ~ 6600 2000
@@
 	0    -1   -1   0
 $EndComp
-Text Label 4500 2450 1    50   ~ 6
+Text Label 4500 2450 1    50   ~ 10
 motor1-
-Text Label 4100 2450 1    50   ~ 6
+Text Label 4100 2450 1    50   ~ 10
 motor1+
 $Comp
@@
 	0    -1   -1   0
 $EndComp
-Text Label 14650 1900 2    50   ~ 6
+Text Label 14650 1900 2    50   ~ 10
 motor1+
-Text Label 14650 1800 2    50   ~ 6
+Text Label 14650 1800 2    50   ~ 10
 motor1-
 Wire Wire Line
@@
 	14450 2450 14450 2500
 Connection ~ 14450 2450
-Text Label 14800 4050 2    50   ~ 6
+Text Label 14800 4050 2    50   ~ 10
 BAT_+
 $Comp
@@
 	14450 4500 14450 4550
 Connection ~ 14450 4500
-Text Label 14800 6100 2    50   ~ 6
+Text Label 14800 6100 2    50   ~ 10
 BAT_+
 $Comp
@@
 	14450 6550 14450 6600
 Connection ~ 14450 6550
-Text Label 14800 8200 2    50   ~ 6
+Text Label 14800 8200 2    50   ~ 10
 BAT_+
 $Comp
@@
 	-1   0    0    1
 $EndComp
-Text Label 2450 5200 2    50   ~ 6
+Text Label 2450 5200 2    50   ~ 10
 B_MCU
 Wire Notes Line
@@
 Wire Notes Line
 	4250 4550 1150 4550
-Text Notes 2750 5200 0    50   ~ 6
+Text Notes 2750 5200 0    50   ~ 10
 Note: On separate in line fuse.
-Text Label 3700 8450 2    50   ~ 6
+Text Label 3700 8450 2    50   ~ 10
 B_MCU
-Text Label 2200 8450 0    50   ~ 6
+Text Label 2200 8450 0    50   ~ 10
 B_MCU
 $Comp
@@
 	11100 1550 11400 1550
 Connection ~ 11400 1550
-Text Label 11100 2550 0    50   ~ 6
+Text Label 11100 2550 0    50   ~ 10
 L_IS_1
 $Comp

Commit message: Ska etsa...
Parts:
- removed C1, C2, C3, C4: CP, Capacitors_THT:CP_Radial_D22.0mm_P10.00mm_SnapIn, symbol Device:C
- removed J6: Motor1_In, TerminalBlocks_Phoenix:TerminalBlock_Phoenix_MKDS1.5-2pol, symbol Connector:Screw_Terminal_01x02
- removed J7: Motor2_In, TerminalBlocks_Phoenix:TerminalBlock_Phoenix_MKDS1.5-2pol, symbol Connector:Screw_Terminal_01x02
- removed J8: Motor3_In, TerminalBlocks_Phoenix:TerminalBlock_Phoenix_MKDS1.5-2pol, symbol Connector:Screw_Terminal_01x02
- removed J9: Motor4_In, TerminalBlocks_Phoenix:TerminalBlock_Phoenix_MKDS1.5-2pol, symbol Connector:Screw_Terminal_01x02
Connections:
- net motor1+: no longer names the net of U1.11 (M+)
- net motor1-: no longer names the net of U1.12 (M-)
- net motor2+: no longer names the net of U2.11 (M+)
- net motor2-: no longer names the net of U2.12 (M-)
- net motor3+: no longer names the net of U3.11 (M+)
- net motor3-: no longer names the net of U3.12 (M-)
- net motor4+: no longer names the net of U4.11 (M+)
- net motor4-: no longer names the net of U4.12 (M-)
- no-connect marks 4 -> 12
Other:
- note removed: "Motor connectors\n"

Commit message: ...
Parts:
- removed C19: CP, Capacitors_THT:CP_Radial_D22.0mm_P10.00mm_SnapIn, symbol Device:CP
Connections:
- net R_EN_1 is gone; now on net L_EN_1: J5.13 (Pin_13), U1.3 (R_EN)
- net R_EN_2 is gone; now on net L_EN_2: J5.25 (Pin_25), U2.3 (R_EN)
- net R_EN_3 is gone; now on net L_EN_3: J5.16 (Pin_16), U3.3 (R_EN)
- net R_EN_4 is gone; now on net L_EN_4: J5.28 (Pin_28), U4.3 (R_EN)
- net LPWM_1: now also J5.9 (Pin_9); no longer J5.11 (Pin_11)
- net LPWM_2: now also J5.21 (Pin_21); no longer J5.23 (Pin_23)
- net LPWM_3: now also J5.20 (Pin_20); no longer J5.18 (Pin_18)
- net LPWM_4: now also J5.32 (Pin_32); no longer J5.30 (Pin_30)
- net L_IS_1: now also J5.31 (Pin_31); no longer J5.19 (Pin_19)
- net L_IS_2: now also J5.19 (Pin_19); no longer J5.31 (Pin_31)
- net L_IS_3: now also J5.22 (Pin_22); no longer J5.10 (Pin_10)
- net L_IS_4: now also J5.10 (Pin_10); no longer J5.22 (Pin_22)
- net RPWM_1: now also J5.11 (Pin_11); no longer J5.9 (Pin_9)
- net RPWM_2: now also J5.23 (Pin_23); no longer J5.21 (Pin_21)
- net RPWM_3: now also J5.18 (Pin_18); no longer J5.20 (Pin_20)
- net RPWM_4: now also J5.30 (Pin_30); no longer J5.32 (Pin_32)
Changed lines of the file:
@@
 Text Label 11100 1550 0    50   ~ 10
 R_IS_1
-Wire Wire Line
-	12600 2100 13250 2100
-Wire Wire Line
-	13250 2000 12600 2000
 $Comp
 L styrenhet-symbols:motor_driver U2
@@
 	2600 10050 2600 10250
 Text Label 3900 9050 2    50   ~ 10
-RPWM_3
+LPWM_3
 Wire Wire Line
 	3900 9050 3250 9050
 Text Label 3900 8950 2    50   ~ 10
-LPWM_3
+RPWM_3
 Wire Wire Line
 	3900 8950 3250 8950
@@
 Text Label 3900 8750 2    50   ~ 10
 L_EN_3
-Text Label 3900 8650 2    50   ~ 10
-R_IS_3
 Text Label 3900 8550 2    50   ~ 10
-L_IS_3
+L_IS_4
 Wire Wire Line
 	3900 8550 3250 8550
@@
 	3250 8850 3900 8850
 Text Label 2100 8550 0    50   ~ 10
-RPWM_1
+LPWM_1
 Wire Wire Line
 	2100 8550 2750 8550
 Text Label 2100 8650 0    50   ~ 10
-LPWM_1
+RPWM_1
 Wire Wire Line
 	2100 8650 2750 8650
@@
 R_IS_1
 Text Label 2100 9050 0    50   ~ 10
-L_IS_1
+L_IS_2
 Wire Wire Line
 	2100 9050 2750 9050
@@
 	2750 8750 2100 8750
 Text Label 2000 9150 0    50   ~ 10
+LPWM_2
+Text Label 2000 9250 0    50   ~ 10
 RPWM_2
-Text Label 2000 9250 0    50   ~ 10
-LPWM_2
 Text Label 2000 9350 0    50   ~ 10
 R_EN_2
@@
 R_IS_2
 Text Label 2000 9650 0    50   ~ 10
-L_IS_2
+L_IS_1
 Text Label 4000 9650 2    50   ~ 10
+LPWM_4
+Text Label 4000 9550 2    50   ~ 10
 RPWM_4
-Text Label 4000 9550 2    50   ~ 10
-LPWM_4
 Text Label 4000 9450 2    50   ~ 10
 R_EN_4
@@
 R_IS_4
 Text Label 4000 9150 2    50   ~ 10
-L_IS_4
+L_IS_3
 Wire Wire Line
 	2600 9950 2600 9850
@@
 Wire Notes Line
 	1150 4300 1150 2900
-$Comp
-L Device:CP C17
-U 1 1 5D24F241
-P 14450 2250
-F 0 "C17" H 14568 2296 50  0000 L CNN
-F 1 "CP" H 14568 2205 50  0000 L CNN
-F 2 "Capacitors_THT:CP_Radial_D22.0mm_P10.00mm_SnapIn" H 14488 2100 50  0001 C CNN
-F 3 "~" H 14450 2250 50  0001 C CNN
-	1    14450 2250
-	1    0    0    -1
-$EndComp
-Wire Wire Line
-	14150 2000 14450 2000
-Wire Wire Line
-	14450 2000 14450 2100
-Connection ~ 14450 2000
-Wire Wire Line
-	14450 2000 14800 2000
 Wire Wire Line
 	14150 2100 14250 2100
@@
 	14250 2450 14450 2450
 Wire Wire Line
-	14450 2450 14450 2400
-Wire Wire Line
 	14450 2450 14450 2500
-Connection ~ 14450 2450
 Text Label 14800 4050 2    50   ~ 10
 BAT_+
@@
 	1    0    0    -1
 $EndComp
-$Comp
-L Device:CP C19
-U 1 1 5D35BBFF
-P 14450 6350
-F 0 "C19" H 14568 6396 50  0000 L CNN
-F 1 "CP" H 14568 6305 50  0000 L CNN
-F 2 "Capacitors_THT:CP_Radial_D22.0mm_P10.00mm_SnapIn" H 14488 6200 50  0001 C CNN
-F 3 "~" H 14450 6350 50  0001 C CNN
-	1    14450 6350
-	1    0    0    -1
-$EndComp
-Wire Wire Line
-	14150 6100 14450 6100
-Wire Wire Line
-	14450 6100 14450 6200
-Connection ~ 14450 6100
-Wire Wire Line
-	14450 6100 14800 6100
 Wire Wire Line
 	14150 6200 14250 6200
@@
 	14250 6550 14450 6550
 Wire Wire Line
-	14450 6550 14450 6500
-Wire Wire Line
 	14450 6550 14450 6600
-Connection ~ 14450 6550
 Text Label 14800 8200 2    50   ~ 10
 BAT_+
@@
 NoConn ~ 14150 8100
 NoConn ~ 14150 8000
+Connection ~ 14450 2450
+Wire Wire Line
+	14450 2450 14450 2400
+Wire Wire Line
+	14450 2000 14800 2000
+Wire Wire Line
+	14150 2000 14450 2000
+Connection ~ 14450 2000
+Wire Wire Line
+	14450 2000 14450 2100
+$Comp
+L Device:CP C17
+U 1 1 5D24F241
+P 14450 2250
+F 0 "C17" H 14568 2296 50  0000 L CNN
+F 1 "CP" H 14568 2205 50  0000 L CNN
+F 2 "Capacitors_THT:CP_Radial_D22.0mm_P10.00mm_SnapIn" H 14488 2100 50  0001 C CNN
+F 3 "~" H 14450 2250 50  0001 C CNN
+	1    14450 2250
+	1    0    0    -1
+$EndComp
+Wire Wire Line
+	14150 6100 14800 6100
+Text Label 3900 8650 2    50   ~ 10
+R_IS_3
+Wire Wire Line
+	12550 2000 13250 2000
+Wire Wire Line
+	12550 2100 12550 2000
+Wire Wire Line
+	12550 2100 13250 2100
+Wire Wire Line
+	12600 4150 12600 4050
+Wire Wire Line
+	12600 6200 12600 6100
+Wire Wire Line
+	12600 8300 12600 8200
 $EndSCHEMATC

Commit message: Update current sense resistor values.
Parts:
- R1, R2, R3, R4, R5, R6, R7, R8: value 440R -> 330R
Changed lines of the file:
@@
 P 11800 1800
 F 0 "R1" H 11730 1754 50  0000 R CNN
-F 1 "440R" H 11730 1845 50  0000 R CNN
+F 1 "330R" H 11730 1845 50  0000 R CNN
 F 2 "Resistors_SMD:R_0603_HandSoldering" V 11730 1800 50  0001 C CNN
 F 3 "~" H 11800 1800 50  0001 C CNN
@@
 P 11800 2800
 F 0 "R2" H 11730 2754 50  0000 R CNN
-F 1 "440R" H 11730 2845 50  0000 R CNN
+F 1 "330R" H 11730 2845 50  0000 R CNN
 F 2 "Resistors_SMD:R_0603_HandSoldering" V 11730 2800 50  0001 C CNN
 F 3 "~" H 11800 2800 50  0001 C CNN
@@
 P 11800 3850
 F 0 "R3" H 11730 3804 50  0000 R CNN
-F 1 "440R" H 11730 3895 50  0000 R CNN
+F 1 "330R" H 11730 3895 50  0000 R CNN
 F 2 "Resistors_SMD:R_0603_HandSoldering" V 11730 3850 50  0001 C CNN
 F 3 "~" H 11800 3850 50  0001 C CNN
@@
 P 11800 4850
 F 0 "R4" H 11730 4804 50  0000 R CNN
-F 1 "440R" H 11730 4895 50  0000 R CNN
+F 1 "330R" H 11730 4895 50  0000 R CNN
 F 2 "Resistors_SMD:R_0603_HandSoldering" V 11730 4850 50  0001 C CNN
 F 3 "~" H 11800 4850 50  0001 C CNN
@@
 P 11800 5900
 F 0 "R5" H 11730 5854 50  0000 R CNN
-F 1 "440R" H 11730 5945 50  0000 R CNN
+F 1 "330R" H 11730 5945 50  0000 R CNN
 F 2 "Resistors_SMD:R_0603_HandSoldering" V 11730 5900 50  0001 C CNN
 F 3 "~" H 11800 5900 50  0001 C CNN
@@
 P 11800 6900
 F 0 "R6" H 11730 6854 50  0000 R CNN
-F 1 "440R" H 11730 6945 50  0000 R CNN
+F 1 "330R" H 11730 6945 50  0000 R CNN
 F 2 "Resistors_SMD:R_0603_HandSoldering" V 11730 6900 50  0001 C CNN
 F 3 "~" H 11800 6900 50  0001 C CNN
@@
 P 11800 7900
 F 0 "R7" H 11730 7854 50  0000 R CNN
-F 1 "440R" H 11730 7945 50  0000 R CNN
+F 1 "330R" H 11730 7945 50  0000 R CNN
 F 2 "Resistors_SMD:R_0603_HandSoldering" V 11730 7900 50  0001 C CNN
 F 3 "~" H 11800 7900 50  0001 C CNN
@@
 P 11800 8900
 F 0 "R8" H 11730 8854 50  0000 R CNN
-F 1 "440R" H 11730 8945 50  0000 R CNN
+F 1 "330R" H 11730 8945 50  0000 R CNN
 F 2 "Resistors_SMD:R_0603_HandSoldering" V 11730 8900 50  0001 C CNN
 F 3 "~" H 11800 8900 50  0001 C CNN
